Commit message: This urdf is updated based on UR5e params on the website. Check descript

File: robots/ur5e/models/ur5-fhdesc2.urdf (robot description, URDF)
Before this commit: robot ur5, 11 links, 10 joints
Links:
- link forearm_link: mass 3.87 -> 2.275
- link shoulder_link: mass 7.778 -> 3.7
- link upper_arm_link: mass 12.93 -> 8.393
- link wrist_1_link: mass 1.96 -> 1.219
- link wrist_2_link: mass 1.96 -> 1.219
- link wrist_3_link: mass 0.202 -> 0.1879
Joints:
- joint ee_fixed_joint: origin xyz=0.0 0.0922 0.0 rpy=0.0 0.0 1.57079632679 -> xyz=0.0 0.0 0.0 rpy=0.0 0.0 1.57079632679
- joint elbow_joint: limit lower=-3.14159265359 upper=3.14159265359 effort=150.0 velocity=3.15 -> lower=-3.14159265359 upper=3.14159265359 effort=150.0 velocity=3.14; origin xyz=0.0 -0.1719 0.612 rpy=0.0 0.0 0.0 -> xyz=0.0 -0.13 0.425 rpy=0.0 0.0 0.0
- joint shoulder_lift_joint: limit lower=-3.14159265359 upper=3.14159265359 effort=330.0 velocity=2.16 -> lower=-6.28318530718 upper=6.28318530718 effort=150.0 velocity=3.14; origin xyz=0.0 0.220941 0.0 rpy=0.0 1.57079632679 0.0 -> xyz=0.0 0.0812 0.0 rpy=0.0 1.57079632679 0.0
- joint shoulder_pan_joint: limit lower=-3.14159265359 upper=3.14159265359 effort=330.0 velocity=2.16 -> lower=-6.28318530718 upper=6.28318530718 effort=150.0 velocity=3.14; origin xyz=0.0 0.0 0.1273 rpy=0.0 0.0 0.0 -> xyz=0.0 0.0 0.1625 rpy=0.0 0.0 0.0
- joint world_joint: origin xyz=0.0 -1.0 1.0 rpy=0.0 0.0 0.0 -> xyz=0.0 0.0 0.0 rpy=0.0 0.0 0.0
- joint wrist_1_joint: limit lower=-3.14159265359 upper=3.14159265359 effort=54.0 velocity=3.2 -> lower=-6.28318530718 upper=6.28318530718 effort=28.0 velocity=6.28; origin xyz=0.0 0.0 0.5723 rpy=0.0 1.57079632679 0.0 -> xyz=0.0 0.0 0.3922 rpy=0.0 1.57079632679 0.0
- joint wrist_2_joint: limit lower=-3.14159265359 upper=3.14159265359 effort=54.0 velocity=3.2 -> lower=-6.28318530718 upper=6.28318530718 effort=28.0 velocity=6.28; origin xyz=0.0 0.1149 0.0 rpy=0.0 0.0 0.0 -> xyz=0.0 0.13 0.0 rpy=0.0 0.0 0.0
- joint wrist_3_joint: limit lower=-3.14159265359 upper=3.14159265359 effort=54.0 velocity=3.2 -> lower=-6.28318530718 upper=6.28318530718 effort=28.0 velocity=6.28; origin xyz=0.0 0.0 0.1157 rpy=0.0 0.0 0.0 -> xyz=0.0 0.0 0.0996 rpy=0.0 0.0 0.0
- joint wrist_3_link-tool0_fixed_joint: origin xyz=0 0.0922 0 rpy=-1.57079632679 0 0 -> xyz=0 0.0822 0 rpy=-1.57079632679 0 0

Commit message: ohh... Finally ikmodel is created for UR5e. Tee is wrong rotation. Fixit

File: robots/ur5e/models/ur5-fhdesc2.urdf (robot description, URDF)
Before this commit: robot ur5e, 11 links, 10 joints
Joints:
- joint world_joint: origin xyz=0.0 0.0 0.0 rpy=0.0 0.0 0.0 -> xyz=0.0 -1.0 -1.0 rpy=0.0 0.0 0.0

Commit message: Tee correct (except for a ridiculous offset in y axis)

File: robots/ur5e/models/ur5-fhdesc2.urdf (robot description, URDF)
Before this commit: robot ur5e, 11 links, 10 joints
Joints:
- joint world_joint: origin xyz=0.0 -1.0 -1.0 rpy=0.0 0.0 0.0 -> xyz=0.0 0.0 0.0 rpy=0.0 0.0 0.0
